Commit message: splitting out wind into separate plugin

File: urdf/wamv_gazebo_dynamics_plugin.xacro (robot description, xacro)
@@ -1,5 +1,5 @@
 <?xml version="1.0"?>
 <robot xmlns:xacro="http://ros.org/wiki/xacro">
-  <xacro:macro name="usv_gazebo" params="name">
+  <xacro:macro name="usv_dynamics_gazebo" params="name">
     <!--Gazebo Plugin for simulating WAM-V dynamics-->
     <gazebo >
