Commit message: reconnecting thrust model

File: urdf/usv_gazebo_dynamics_plugin.xacro (robot description, xacro)
@@ -1,5 +1,5 @@
 <?xml version="1.0"?>
 <robot xmlns:xacro="http://ros.org/wiki/xacro">
-  <xacro:macro name="usv_gazebo" params="name">
+  <xacro:macro name="usv_dynamics_gazebo" params="name">
     <!--Gazebo Plugin for simulating Kingfisher dynamics-->
     <gazebo >

File: urdf/wamv_gazebo_thrust_plugin.xacro (robot description, xacro)
@@ -5,5 +5,5 @@
     <gazebo >
       <plugin name="usv_thrust_${name}" filename="libusv_gazebo_thrust_plugin.so">
-	<bodyName>base_link</bodyName>
+	<bodyName>base_footprint</bodyName>
 	<!-- Which thruster curve to use -->
 	<mappingType>1</mappingType>
